Commit message: feat: include teleop.launch

File: slam_project/urdf/udacity_bot.xacro (robot description, xacro)
@@ -143,5 +143,5 @@
       <origin xyz="0 0 0" rpy=" 0 0 0"/>
       <geometry>
-	<mesh filename="package://sweeping_bot/meshes/kinect.dae"/>
+	<mesh filename="package://slam_project/meshes/kinect.dae"/>
       </geometry>
     </visual>

Commit message: fix: update urdfs udacity_bot

File: slam_project/urdf/udacity_bot.xacro (robot description, xacro)
@@ -119,12 +119,8 @@
     <dynamics damping="1.0" friction="1.0"/>
   </joint>
-  <joint type="fixed" name="camera_joint">
-    <origin xyz="0.2 0 0" rpy="0 0 0"/>
-    <child link="camera"/>
-    <parent link="chassis"/>
-  </joint>
-  <link name='camera'>
+  <link name='camera_rgb_frame'>
+   <pose>0 0 0.1 0 0 0</pose>
     <inertial>
-      <mass value="0.1"/>
+      <mass value="0.564"/>
       <origin xyz="0 0 0" rpy=" 0 0 0"/>
       <inertia
@@ -147,10 +143,29 @@
     </visual>
   </link>
-  <joint type="fixed" name="hokuyo_joint">
-    <origin xyz="0.15 0 0.1" rpy="0 0 0"/>
-    <child link="hokuyo"/>
+ <joint type="fixed" name="camera_rgb_frame_joint">
+    <origin xyz="0.2 0 0" rpy="0 0 0"/>
+    <child link="camera_rgb_frame"/>
     <parent link="chassis"/>
   </joint>
+  <link name="camera_rgb_optical_frame"/>
+  <joint name="camera_rgb_optical_joint" type="fixed">
+    <origin xyz="0 0 0" rpy="-1.571 0 -1.571"/>
+    <parent link="camera_rgb_frame"/>
+    <child link="camera_rgb_optical_frame"/>
+  </joint>
+  <link name="camera_depth_frame"/>
+  <joint name="camera_depth_joint" type="fixed">
+    <origin xyz="0 0 0" rpy="0 0 0"/>
+    <parent link="camera_rgb_frame"/>
+    <child link="camera_depth_frame"/>
+  </joint>
+  <link name="camera_depth_optical_frame"/>
+  <joint name="camera_depth_optical_joint" type="fixed">
+    <origin xyz="0 0 0" rpy="-1.571 0 -1.571"/>
+    <parent link="camera_depth_frame"/>
+    <child link="camera_depth_optical_frame"/>
+  </joint>
   <link name='hokuyo'>
+  <pose>0 0 0.1 0 0 0</pose>
     <inertial>
       <mass value="0.1"/>
@@ -175,3 +190,8 @@
     </visual>
   </link>
+  <joint type="fixed" name="hokuyo_joint">
+    <origin xyz="0.15 0 0.1" rpy="0 0 0"/>
+    <child link="hokuyo"/>
+    <parent link="chassis"/>
+  </joint>
 </robot>

Commit message: feat: complete the project

File: slam_project/urdf/udacity_bot.xacro (robot description, xacro)
@@ -119,5 +119,5 @@
     <dynamics damping="1.0" friction="1.0"/>
   </joint>
-  <link name='camera_rgb_frame'>
+  <link name='camera_rgb'>
    <pose>0 0 0.1 0 0 0</pose>
     <inertial>
@@ -143,7 +143,7 @@
     </visual>
   </link>
- <joint type="fixed" name="camera_rgb_frame_joint">
+ <joint type="fixed" name="camera_rgb_joint">
     <origin xyz="0.2 0 0" rpy="0 0 0"/>
-    <child link="camera_rgb_frame"/>
+    <child link="camera_rgb"/>
     <parent link="chassis"/>
   </joint>
@@ -151,17 +151,17 @@
   <joint name="camera_rgb_optical_joint" type="fixed">
     <origin xyz="0 0 0" rpy="-1.571 0 -1.571"/>
-    <parent link="camera_rgb_frame"/>
+    <parent link="camera_rgb"/>
     <child link="camera_rgb_optical_frame"/>
   </joint>
-  <link name="camera_depth_frame"/>
+  <link name="camera_depth"/>
   <joint name="camera_depth_joint" type="fixed">
     <origin xyz="0 0 0" rpy="0 0 0"/>
-    <parent link="camera_rgb_frame"/>
-    <child link="camera_depth_frame"/>
+    <parent link="camera_rgb"/>
+    <child link="camera_depth"/>
   </joint>
   <link name="camera_depth_optical_frame"/>
   <joint name="camera_depth_optical_joint" type="fixed">
     <origin xyz="0 0 0" rpy="-1.571 0 -1.571"/>
-    <parent link="camera_depth_frame"/>
+    <parent link="camera_depth"/>
     <child link="camera_depth_optical_frame"/>
   </joint>
